File: hardware/PC02/PC02.brd (EAGLE design)
At the start: 71.4 x 54.6 mm, 9 parts, among them J1 HEADER_1X23, J13 HEADER_1X8, J14 HEADER_1X8, J15 HEADER_1X8, J16 HEADER_1X8, J2 HEADER_1X23, J3 HEADER_1X23, J4 HEADER_1X23

Commit message: added 2 mounting holes
Parts:
- added U$1, U$3: (no value), microbuilder:MOUNTINGHOLE_3.0_PLATEDTHIN
Other:
- outline, holes or cut-outs redrawn

Commit message: Version PC02
Other:
- outline, holes or cut-outs redrawn
