File: hardware/PC02/PC02.sch (EAGLE design)
At the start: 9 parts, among them J1 HEADER_1X23, J13 HEADER_1X8, J14 HEADER_1X8, J15 HEADER_1X8, J16 HEADER_1X8, J2 HEADER_1X23, J3 HEADER_1X23, J4 HEADER_1X23

Commit message: Version PC02
Other:
- note added: "A. HIAM / T. PRICE"
- note added: "lgx.co / smokedprojects.blogspot.com"
- note removed: "A. HIAM"
- note removed: "lgx.co"
Changed lines of the file:
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@@
 <sheet>
 <plain>
-<text x="185.42" y="-15.24" size="2.1844" layer="97" font="vector">A. HIAM</text>
+<text x="185.42" y="-15.24" size="2.1844" layer="97" font="vector">A. HIAM / T. PRICE</text>
 <text x="180.34" y="-10.16" size="2.1844" layer="97" font="vector">PC01</text>
 <text x="251.46" y="-10.16" size="2.1844" layer="97" font="vector">1</text>
-<text x="180.34" y="-20.32" size="2.1844" layer="97" font="vector">lgx.co</text>
+<text x="180.34" y="-20.32" size="2.1844" layer="97" font="vector">lgx.co / smokedprojects.blogspot.com</text>
 <text x="170.18" y="-25.4" size="2.1844" layer="97" font="vector">CC BY 3.0</text>
 </plain>
